File: ql_Cumana.kicad_sch (KiCad schematic)
At the start: 40 parts, among them J1 QL_SLOT_DIN41612_CARD, J2 Conn_02x17_Odd_Even, U1 LS04, U10 74LS273, U11 74LS133, U12 FDC_WD1772, U13 27C128, U14 74LS245, U2 7805, U3 LS00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

Commit message: Initial
Parts:
- C12: value 27p -> 100n
- C4: now fitted
Connections:
- net A4: now also U11.12
- net A5: now also U11.13
- net A6: now also U11.14
- net A7: now also U11.15
- net GND: now also U8.5
- net ROM_OE: now also U3.10
- net FDREG_CS: now reaches U10.11 (Cp), U3.8
- net PGM renamed VCC_r
- no-connect marks 28 -> 29
Other:
- note removed: "1 2 3 4"
- note removed: "XT MODE: 2-3 (Plain Cable , drives DS0, DS1) AT MODE: 1-2, 3-4 (Cross Cable, both drives DS1)"
- note removed: "normal: 1 & 2, 3 & 4, - DS0 is DS0 and DS1 is DS1 inverse: 1 & 3, 2 & 4 - DS0 is DS1 and DS1 is DS0"
- title: CST Q-Disc Interface Version 4 -> Cumana Disc Interface
- moved on the sheet: U11B, U1G, U3A, U3B, U3C, U3E, U5A, U5C, U6A, U6B, U6F, U6G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
