File: ql_Cumana.kicad_sch (KiCad schematic)
At the start: 40 parts, among them J1 QL_SLOT_DIN41612_CARD, J2 Conn_02x17_Odd_Even, U1 LS04, U10 74LS273, U11 74LS133, U12 FDC_WD1772, U13 27C128, U14 74LS245, U2 7805, U3 LS00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

Commit message: update silkscreen
Parts:
- renumbered Y1 to X1
Changed lines of the file:
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@@
 	(wire
 		(pts
-			(xy 118.11 68.58) (xy 116.84 68.58)
+			(xy 116.84 68.58) (xy 128.27 68.58)
 		)
 		(stroke
@@
 	(wire
 		(pts
-			(xy 128.27 68.58) (xy 118.11 68.58)
-		)
-		(stroke
-			(width 0)
-			(type default)
-		)
-	)
-	(wire
-		(pts
 			(xy 180.34 115.57) (xy 200.66 115.57)
 		)
@@
 		(on_board yes)
 		(dnp no)
-		(property "Reference" "Y1"
+		(property "Reference" "X1"
 			(at 332.74 180.34 0)
 			(effects
@@
 			(project "ql_Cumana"
 				(path "/aecd9f77-969e-41c8-a7ad-8348a70f1d7d"
-					(reference "Y1")
+					(reference "X1")
 					(unit 1)
 				)

Commit message: update component values
Parts:
- R2: value 3K7 -> 4K7
- TR1: value BC2369 -> 2N2369
- U1: value LS04 -> 74LS04
- U3: value LS00 -> 74LS00
- U7, U8: value 74LS16 -> 74LS06
Changed lines of the file:
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@@
 			)
 		)
-		(property "Value" "74LS16"
+		(property "Value" "74LS06"
 			(at 293.37 78.105 0)
 			(effects
@@
 			)
 		)
-		(property "Value" "74LS16"
+		(property "Value" "74LS06"
 			(at 267.97 139.065 0)
 			(effects
@@
 			)
 		)
-		(property "Value" "LS00"
+		(property "Value" "74LS00"
 			(at 43.18 210.82 0)
 			(effects
@@
 			)
 		)
-		(property "Value" "74LS16"
+		(property "Value" "74LS06"
 			(at 267.97 109.22 0)
 			(effects
@@
 			)
 		)
-		(property "Value" "LS00"
+		(property "Value" "74LS00"
 			(at 247.65 188.595 0)
 			(effects
@@
 			)
 		)
-		(property "Value" "LS04"
+		(property "Value" "74LS04"
 			(at 321.31 193.04 0)
 			(effects
@@
 			)
 		)
-		(property "Value" "BC2369"
+		(property "Value" "2N2369"
 			(at 102.87 184.1499 0)
 			(effects
@@
 			)
 		)
-		(property "Value" "LS04"
+		(property "Value" "74LS04"
 			(at 285.75 257.81 0)
 			(effects
@@
 			)
 		)
-		(property "Value" "3K7"
+		(property "Value" "4K7"
 			(at 344.678 204.724 90)
 			(effects
@@
 			)
 		)
-		(property "Value" "LS04"
+		(property "Value" "74LS04"
 			(at 176.53 266.7 0)
 			(effects
@@
 			)
 		)
-		(property "Value" "LS04"
+		(property "Value" "74LS04"
 			(at 125.73 97.79 0)
 			(effects
@@
 			)
 		)
-		(property "Value" "LS04"
+		(property "Value" "74LS04"
 			(at 285.75 280.67 0)
 			(effects
@@
 			)
 		)
-		(property "Value" "74LS16"
+		(property "Value" "74LS06"
 			(at 280.67 116.84 0)
 			(effects
@@
 			)
 		)
-		(property "Value" "74LS16"
+		(property "Value" "74LS06"
 			(at 267.97 124.46 0)
 			(effects
@@
 			)
 		)
-		(property "Value" "74LS16"
+		(property "Value" "74LS06"
 			(at 280.67 132.715 0)
 			(effects
@@
 			)
 		)
-		(property "Value" "74LS16"
+		(property "Value" "74LS06"
 			(at 281.94 69.85 0)
 			(effects
@@
 			)
 		)
-		(property "Value" "74LS16"
+		(property "Value" "74LS06"
 			(at 280.67 101.6 0)
 			(effects
@@
 			)
 		)
-		(property "Value" "74LS16"
+		(property "Value" "74LS06"
 			(at 201.295 265.43 0)
 			(effects
@@
 			)
 		)
-		(property "Value" "LS00"
+		(property "Value" "74LS00"
 			(at 247.65 206.375 0)
 			(effects
@@
 			)
 		)
-		(property "Value" "74LS16"
+		(property "Value" "74LS06"
 			(at 215.265 265.43 0)
 			(effects
@@
 			)
 		)
-		(property "Value" "LS04"
+		(property "Value" "74LS04"
 			(at 285.75 269.24 0)
 			(effects
@@
 			)
 		)
-		(property "Value" "LS00"
+		(property "Value" "74LS00"
 			(at 135.89 214.63 0)
 			(effects
@@
 			)
 		)
-		(property "Value" "LS04"
+		(property "Value" "74LS04"
 			(at 350.52 193.04 0)
 			(effects
@@
 			)
 		)
-		(property "Value" "74LS16"
+		(property "Value" "74LS06"
 			(at 212.09 229.87 0)
 			(effects
@@
 			)
 		)
-		(property "Value" "74LS16"
+		(property "Value" "74LS06"
 			(at 281.94 85.725 0)
 			(effects
@@
 			)
 		)
-		(property "Value" "74LS16"
+		(property "Value" "74LS06"
 			(at 283.21 234.95 0)
 			(effects
@@
 			)
 		)
-		(property "Value" "LS00"
+		(property "Value" "74LS00"
 			(at 191.77 265.43 0)
 			(effects
@@
 			)
 		)
-		(property "Value" "74LS16"
+		(property "Value" "74LS06"
 			(at 293.37 60.96 0)
 			(effects

Commit message: complete
Parts:
- U12: value FDC_WD1772 -> FDC_WD1770
Changed lines of the file:
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@@
 			)
 		)
-		(property "Value" "FDC_WD1772"
+		(property "Value" "FDC_WD1770"
 			(at 232.41 59.69 0)
 			(effects
