File: ql_Cumana.kicad_pcb (KiCad board)
At the start: 2 copper layers, 129.5 x 100 mm, 40 parts, among them J1 QL_SLOT_DIN41612_CARD, J2 Conn_02x17_Odd_Even, U1 74LS04, U10 74LS273, U11 74LS133, U12 FDC_WD1772, U13 27C128, U14 74LS245, U2 7805, U3 74LS00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

Commit message: complete
Parts:
- U12: value FDC_WD1772 -> FDC_WD1770
Routing:
- net +5V: track 521.8 -> 524.0 mm
- net /VCC_r: track 134.6 -> 134.0 mm
Changed lines of the file:
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@@
 	(paper "A4")
 	(title_block
-		(title "CST Q-Disc Interface Version 4")
-		(date "2023-05-20")
+		(title "CUMANA Disc Interface")
+		(date "2026-03-28")
 		(rev "00")
 		(company "Repro by Alvaro Alea Fdz.")
-		(comment 1 "to use with ROM Version 1.18")
-		(comment 2 "Disc Interface for Sinclair QL")
+		(comment 1 "Disc Interface for Sinclair QL")
 	)
 	(layers
@@
 			)
 		)
-		(property "Value" "FDC_WD1772"
+		(property "Value" "FDC_WD1770"
 			(at 7.62 35.35 90)
 			(layer "F.Fab")
@@
 		(layer "User.1")
 		(pts
-			(xy 197.632 143.823) (xy 197.632 43.873)
+			(xy 197.612 143.823) (xy 197.612 43.873)
 		)
 		(height 8.89)
@@
 		)
 		(gr_text "99,9500 mm"
-			(at 205.372 93.848 90)
+			(at 205.352 93.848 90)
 			(layer "User.1")
 			(effects
@@
 		(layer "User.1")
 		(pts
-			(xy 197.632 49.398) (xy 197.632 43.873)
+			(xy 197.632 49.398) (xy 197.612 43.873)
 		)
 		(height 2.5)
@@
 		(layer "User.1")
 		(pts
-			(xy 197.632 143.823) (xy 197.632 138.298)
+			(xy 197.612 143.823) (xy 197.612 138.298)
 		)
 		(height 2.5)
@@
 		)
 		(gr_text "5,5250 mm"
-			(at 198.532 141.0605 90)
+			(at 198.512 141.0605 90)
 			(layer "User.1")
 			(effects
@@
 	)
 	(segment
-		(start 144.272 110.998)
-		(end 144.272 107.823)
-		(width 0.75)
-		(layer "F.Cu")
-		(net 1)
-	)
-	(segment
-		(start 83.947 142.113)
-		(end 78.867 137.033)
+		(start 114.427 142.113)
+		(end 83.185 142.24)
 		(width 1)
 		(layer "F.Cu")
@@
 	)
 	(segment
-		(start 114.427 142.113)
-		(end 83.947 142.113)
-		(width 1)
+		(start 144.272 110.998)
+		(end 144.272 107.823)
+		(width 0.75)
 		(layer "F.Cu")
 		(net 1)
@@
 	)
 	(segment
+		(start 78.867 137.287)
+		(end 78.867 131.953)
+		(width 1)
+		(layer "F.Cu")
+		(net 1)
+	)
+	(segment
 		(start 146.812 65.913)
 		(end 145.542 64.643)
@@
 	)
 	(segment
+		(start 83.185 142.24)
+		(end 78.867 137.287)
+		(width 1)
+		(layer "F.Cu")
+		(net 1)
+	)
+	(segment
 		(start 78.867 131.953)
 		(end 78.867 131.318)
@@
 	)
 	(segment
-		(start 78.867 137.033)
-		(end 78.867 131.953)
-		(width 1)
-		(layer "F.Cu")
-		(net 1)
-	)
-	(segment
 		(start 130.302 44.958)
 		(end 149.987 44.958)
@@
 		(drill 0.8)
 		(layers "F.Cu" "B.Cu")
-		(tenting front back)
+		(tenting none)
 		(net 1)
 	)
@@
 		(drill 0.8)
 		(layers "F.Cu" "B.Cu")
-		(tenting front back)
+		(tenting none)
 		(net 1)
 	)
@@
 	)
 	(segment
-		(start 130.302 90.043)
-		(end 129.667 90.043)
-		(width 0.75)
-		(layer "B.Cu")
-		(net 1)
-	)
-	(segment
 		(start 86.487 55.118)
 		(end 91.567 55.118)
@@
 	)
 	(segment
-		(start 129.667 90.043)
-		(end 127.127 90.043)
+		(start 127.127 90.043)
+		(end 131.572 90.043)
 		(width 0.75)
 		(layer "B.Cu")
@@
 	)
 	(segment
-		(start 131.572 90.043)
-		(end 129.667 90.043)
-		(width 0.75)
-		(layer "B.Cu")
-		(net 1)
-	)
-	(segment
 		(start 110.617 63.373)
 		(end 79.582 63.373)
@@
 		(start 122.738 104.704)
 		(end 122.738 110.307)
-		(width 1)
+		(width 0.75)
 		(layer "F.Cu")
 		(net 81)
@@
 		(start 118.872 131.953)
 		(end 118.872 128.949174)
-		(width 1)
+		(width 0.5)
 		(layer "F.Cu")
 		(net 81)
@@
 		(start 121.412 103.378)
 		(end 122.738 104.704)
-		(width 1)
+		(width 0.75)
 		(layer "F.Cu")
 		(net 81)
@@
 		(start 120.777 112.268)
 		(end 122.738 110.307)
-		(width 1)
+		(width 0.75)
 		(layer "F.Cu")
 		(net 81)
@@
 		(start 123.952 119.253)
 		(end 120.777 116.078)
-		(width 1)
+		(width 0.75)
 		(layer "F.Cu")
 		(net 81)
@@
 		(start 123.952 121.793)
 		(end 123.952 119.253)
-		(width 1)
+		(width 0.75)
 		(layer "F.Cu")
 		(net 81)
@@
 		(start 120.777 116.078)
 		(end 120.777 112.268)
-		(width 1)
+		(width 0.75)
 		(layer "F.Cu")
 		(net 81)
@@
 		(start 118.872 128.949174)
 		(end 120.948174 126.873)
-		(width 1)
+		(width 0.5)
 		(layer "F.Cu")
 		(net 81)
@@
 		(start 123.952 137.033)
 		(end 118.872 131.953)
-		(width 1)
+		(width 0.5)
 		(layer "F.Cu")
 		(net 81)
@@
 		(start 120.948174 126.873)
 		(end 123.317 126.873)
-		(width 1)
+		(width 0.5)
 		(layer "F.Cu")
 		(net 81)
@@
 	)
 	(segment
-		(start 87.757 105.283)
-		(end 91.567 105.283)
-		(width 1)
-		(layer "B.Cu")
-		(net 81)
-	)
-	(segment
 		(start 102.997 66.548)
 		(end 100.497 66.548)
@@
 	)
 	(segment
-		(start 121.412 105.334)
-		(end 91.618 105.334)
-		(width 1)
-		(layer "B.Cu")
-		(net 81)
-	)
-	(segment
 		(start 78.867 50.038)
 		(end 78.867 52.578)
@@
 	)
 	(segment
+		(start 93.091 105.459)
+		(end 87.581 105.459)
+		(width 1)
+		(layer "B.Cu")
+		(net 81)
+	)
+	(segment
 		(start 91.527 67.858)
 		(end 90.297 69.088)
@@
 	)
 	(segment
-		(start 91.618 105.334)
-		(end 91.567 105.283)
+		(start 87.581 105.459)
+		(end 87.0585 105.9815)
 		(width 1)
 		(layer "B.Cu")
@@
 	)
 	(segment
+		(start 121.287 105.459)
+		(end 119.507 105.459)
+		(width 1)
+		(layer "B.Cu")
+		(net 81)
+	)
+	(segment
 		(start 80.137 117.348)
 		(end 77.597 117.348)
@@
 	)
 	(segment
+		(start 119.507 105.459)
+		(end 126.316 105.459)
+		(width 1)
+		(layer "B.Cu")
+		(net 81)
+	)
+	(segment
 		(start 78.867 48.133)
 		(end 107.442 48.133)
@@
 	)
 	(segment
-		(start 126.441 105.334)
-		(end 121.412 105.334)
+		(start 123.317 128.778)
+		(end 141.097 128.778)
 		(width 1)
 		(layer "B.Cu")
@@
 	)
 	(segment
-		(start 123.317 128.778)
-		(end 141.097 128.778)
+		(start 91.743 105.459)
+		(end 91.567 105.283)
 		(width 1)
 		(layer "B.Cu")
@@
 	)
 	(segment
-		(start 135.382 55.118)
-		(end 141.732 55.118)
+		(start 121.412 105.334)
+		(end 121.287 105.459)
 		(width 1)
 		(layer "B.Cu")
@@
 	)
 	(segment
-		(start 126.492 105.283)
-		(end 126.441 105.334)
+		(start 135.382 55.118)
+		(end 141.732 55.118)
 		(width 1)
 		(layer "B.Cu")
@@
 	)
 	(segment
-		(start 87.757 106.633)
-		(end 87.757 105.283)
+		(start 126.316 105.459)
+		(end 126.492 105.283)
 		(width 1)
 		(layer "B.Cu")
@@
 	)
 	(segment
+		(start 119.507 105.459)
+		(end 93.091 105.459)
+		(width 1)
+		(layer "B.Cu")
+		(net 81)
+	)
+	(segment
 		(start 111.887 52.578)
 		(end 111.887 59.563)
@@
 	)
 	(segment
-		(start 87.757 105.283)
+		(start 93.091 105.459)
+		(end 91.743 105.459)
+		(width 1)
+		(layer "B.Cu")
+		(net 81)
+	)
+	(segment
+		(start 87.0585 105.9815)
 		(end 77.597 115.443)
 		(width 1)
@@
 	)
 	(segment
-		(start 155.702 46.863)
-		(end 151.892 46.863)
+		(start 151.892 46.863)
+		(end 173.482 46.863)
 		(width 0.35)
 		(layer "F.Cu")
@@
 	)
 	(segment
-		(start 155.702 46.863)
-		(end 155.067 46.863)
-		(width 0.35)
-		(layer "F.Cu")
-		(net 136)
-	)
-	(segment
 		(start 150.622 48.133)
 		(end 148.082 48.133)
 		(width 0.35)
 		(layer "F.Cu")
-		(net 136)
-	)
-	(segment
-		(start 155.702 46.863)
-		(end 173.482 46.863)
-		(width 0.35)
-		(layer "F.Cu")
